File: iNode/Devesh/HWBDSN/sensor_node.kicad_pcb (KiCad board)
At the start: 2 copper layers, 90.3 x 33.2 mm, 47 parts, among them J102 Conn_01x01, J103 Conn_01x02, J105 extenal_battery, SW101 SW_Push, U1 CC110L, U101 ATtiny1606-M, U2 PIR_digital_sensor, U3 PIR_digital_sensor, Y1 26MHz Crystal, 10pF

Commit message: Add files via upload
Parts:
- removed BT1: Battery_Cell, Battery:BatteryHolder_LINX_BAT-HLD-012-SMT
- removed J103: Conn_01x02, Connector_PinHeader_2.54mm:PinHeader_1x02_P2.54mm_Vertical
- removed R105, R106: 10K, Resistor_SMD:R_0603_1608Metric
- added C101: 0.1uF, 10V, Capacitor_SMD:C_0402_1005Metric, F.Cu at (141.2, 125.9)
- J105: footprint Connector_PinHeader_2.54mm:PinHeader_1x02_P2.54mm_Vertical -> Connector_JST:JST_EH_B2B-EH-A_1x02_P2.50mm_Vertical
- U2: moved to B.Cu
- moved J102 11.2 mm to (137.7, 141.9)
- moved R3 8.63 mm to (126.5, 129.4)
- moved U3 5.46 mm to (128.6, 120.6), turned to 270 degrees
- moved U2 5.12 mm to (128.5, 139.4)
- moved D101 3.60 mm to (141.4, 117.9)
- moved D102 3.60 mm to (139.7, 117.9)
- moved D103 3.60 mm to (138.0, 117.9)
- moved R102 3.60 mm to (141.4, 120.9)
- moved R103 3.60 mm to (139.7, 120.9)
- moved R104 3.60 mm to (138.0, 120.9)
- moved J105 1.52 mm to (150.1, 119.0), turned to 0 degrees
- renumbered LDR to R3
Routing:
- net +3V3: track 121.1 -> 106.1 mm, vias 11 -> 9
- net /Sheet5FFE69EF/LDR: track 36.8 -> 28.2 mm
- net /Sheet6001F810/SDA: track 6.20 -> 0.00 mm
- net /Sheet6001F810/SCL: track 5.96 -> 0.00 mm
- net /Sheet6001F810/RESETn_UPDI: track 19.6 -> 24.6 mm
- net /Sheet5FFE69EF/PIR_1: track 19.7 -> 24.3 mm, vias 1 -> 0
- net /Sheet6001F810/RED: track 6.66 -> 4.24 mm
- net /Sheet6001F837/CSn: track 18.9 -> 21.2 mm
- net GND: track 15.5 -> 17.5 mm, vias 40 -> 55
- net /Sheet6001F810/YELLOW: track 5.71 -> 3.74 mm
- net /Sheet6001F810/GREEN: track 4.39 -> 3.27 mm
- net /Sheet5FFE69EF/PIR_2: track 14.2 -> 13.6 mm
Other:
- board size 90.3 x 33.2 mm -> 57.1 x 28.8 mm
- board text removed: "SCL"
- board text removed: "SDA"
